Commit message: update static urdf

File: maxwell_defs/urdf/maxwell.urdf (robot description, URDF)
Before this commit: robot maxwell, 48 links, 47 joints
Links:
- added link arm_upperarm_roll_link, mass 0.00001; collision box size=0.0762 0.053 0.044; visual mesh filename=package://maxwell_defs/meshes/sixdof_bracket1.stl scale=0.001 0.001 0.001
- added link arm_upperarm_roll_servo_link, mass 0.00001; collision box size=0.0611 0.0470 0.0420; visual mesh filename=package://maxwell_defs/meshes/rx64.stl scale=1 1 1
- link arm_shoulder_lift_link: geometry collision box size=0.0762 0.053 0.044; visual mesh filename=package://maxwell_defs/meshes/sixdof_bracket2.stl scale=0.001 0.001 0.001
Joints:
- added joint arm_upperarm_roll_joint: type revolute, parent arm_upperarm_roll_servo_link, child arm_upperarm_roll_link, origin xyz=0 0 0 rpy=-1.57 0 1.57, axis 1 0 0, limit lower=-3.14 upper=3.14 effort=30 velocity=0.524
- added joint arm_upperarm_roll_servo_joint: type fixed, parent arm_shoulder_lift_link, child arm_upperarm_roll_servo_link, origin xyz=0.0839978 0 0 rpy=1.57 1.57 0
- joint arm_elbow_flex_joint: origin xyz=0.16 0 0 rpy=0 0 0 -> xyz=0.074295 0 0 rpy=0 0 0; parent arm_shoulder_lift_link -> arm_upperarm_roll_link

Commit message: update exported urdf

File: maxwell_defs/urdf/maxwell.urdf (robot description, URDF)
Before this commit: robot maxwell, 50 links, 49 joints
Links:
- link arm_shoulder_lift_link: geometry collision box size=0.0762 0.053 0.044; visual mesh filename=package://maxwell_defs/meshes/sixdof_bracket1.stl scale=0.001 0.001 0.001
- link arm_upperarm_roll_link: geometry collision box size=0.0762 0.053 0.044; visual mesh filename=package://maxwell_defs/meshes/sixdof_bracket2.stl scale=0.001 0.001 0.001
Joints:
- joint arm_elbow_flex_joint: origin xyz=0.074295 0 0 rpy=0 0 0 -> xyz=0.0869955 0 0 rpy=0 0 0
- joint arm_upperarm_roll_joint: limit lower=-3.14 upper=3.14 effort=30 velocity=0.524 -> lower=-2 upper=2 effort=30 velocity=0.524
- joint arm_upperarm_roll_servo_joint: origin xyz=0.0839978 0 0 rpy=1.57 1.57 0 -> xyz=0.0712978 0 0 rpy=1.57 1.57 0

Commit message: update moveit config

File: maxwell_defs/urdf/maxwell.urdf (robot description, URDF)
Before this commit: robot maxwell, 50 links, 49 joints
Links:
- removed link gripper_link
Joints:
- removed joint gripper_joint
- joint arm_wrist_roll_joint: origin xyz=0.031 0 0 rpy=0 0 0 -> xyz=0.041 0 0 rpy=0 0 0
