Commit message: temporary branch with short, armless maxwell

File: maxwell_defs/urdf/maxwell.urdf.xacro (robot description, xacro)
@@ -1,6 +1,6 @@
 <?xml version="1.0"?>
 <robot xmlns:xacro="http://www.ros.org/wiki/xacro" name="maxwell">
-  <xacro:property name="arm_height" value="0.6604"/> <!-- deck to arm_link at max height-->
-  <xacro:property name="column_height" value="1.172775" /> <!-- deck to top of 80/20 -->
+  <xacro:property name="arm_height" value="0.2"/> <!-- deck to arm_link at max height-->
+  <xacro:property name="column_height" value="0.258375" /> <!-- deck to top of 80/20 -->
   <xacro:include filename="$(find maxwell_defs)/urdf/hardware/ax12.xacro" />
   <xacro:include filename="$(find maxwell_defs)/urdf/hardware/rx64.xacro" />
@@ -9,6 +9,4 @@
   <xacro:include filename="$(find maxwell_defs)/urdf/base.urdf.xacro" />
   <xacro:include filename="$(find maxwell_defs)/urdf/torso.urdf.xacro" />
-  <xacro:include filename="$(find maxwell_defs)/urdf/arm.urdf.xacro" />
-  <xacro:include filename="$(find maxwell_defs)/urdf/gripper.urdf.xacro" />
   <xacro:include filename="$(find maxwell_defs)/urdf/head.urdf.xacro" />
   <xacro:include filename="$(find maxwell_defs)/urdf/materials.urdf.xacro" />
@@ -19,21 +17,4 @@
     <origin xyz="-0.00635 0 ${base_size_z+arm_height}" rpy="0 0 0"/>
   </maxwell_torso>
-  <!-- Live joint between torso and arm -->
-  <joint name="arm_lift_joint" type="prismatic">
-    <axis xyz="0 0 1" />
-    <limit lower="-0.464" upper="0" effort="30" velocity="0.0508"/>
-    <origin xyz="0 0 0" rpy="0 0 0" />
-    <parent link="torso_link"/>
-    <child link="arm_lift_link"/>
-  </joint>
-  <link name="arm_lift_link"/>
-  <!-- Arm -->
-  <maxwell_arm name="arm" parent="arm_lift_link">
-    <origin xyz="0.0611 0 0" rpy="0 0 0"/>
-  </maxwell_arm>
-  <!-- Gripper -->
-  <maxwell_gripper name="gripper" parent="arm_wrist_roll" color="Orange">
-    <origin xyz="0 0 0" rpy="0 0 0" />
-  </maxwell_gripper>
   <!-- Head -->
   <maxwell_head name="head" parent="torso_link" color="Orange">

File: maxwell_defs/urdf/torso.urdf.xacro (robot description, xacro)
@@ -22,24 +22,4 @@
       </collision>
     </link>
-    <joint name="${name}_actuator_joint" type="fixed">
-      <origin xyz="0 0 0" rpy="0 0 0"/>
-      <parent link="${name}_link"/>
-      <child link="${name}_actuator_link"/>
-    </joint>
-    <link name="${name}_actuator_link">
-      <visual>
-        <origin xyz="-0.05 -0.0127 -0.560" rpy="0 0 3.14" />
-        <geometry>
-          <mesh filename="package://maxwell_defs/meshes/FA-35-TR.stl" scale="0.001 0.001 0.001"/>
-        </geometry>
-        <material name="Grey"/>
-      </visual>
-      <collision>
-        <origin xyz="-0.03 0 ${-0.650/2+.08}" rpy="0 0 0 " />
-        <geometry>
-          <box size="0.03 0.0254 0.650"/>
-        </geometry>
-      </collision>
-    </link>
   </macro>
 </robot>

Commit message: update URDF for parallel gripper

File: maxwell_defs/urdf/maxwell.urdf.xacro (robot description, xacro)
@@ -11,4 +11,5 @@
   <xacro:include filename="$(find maxwell_defs)/urdf/arm.urdf.xacro" />
   <xacro:include filename="$(find maxwell_defs)/urdf/gripper.urdf.xacro" />
+  <xacro:include filename="$(find maxwell_defs)/urdf/parallel_gripper.urdf.xacro" />
   <xacro:include filename="$(find maxwell_defs)/urdf/head.urdf.xacro" />
   <xacro:include filename="$(find maxwell_defs)/urdf/materials.urdf.xacro" />
@@ -32,8 +33,16 @@
     <origin xyz="0.0611 0 0" rpy="0 0 0"/>
   </maxwell_arm>
-  <!-- Gripper -->
-  <maxwell_gripper name="gripper" parent="arm_wrist_roll" color="Orange">
-    <origin xyz="0 0 0" rpy="0 0 0" />
-  </maxwell_gripper>
+  <!-- Older Two Finger Gripper -->
+  <xacro:unless value="$(arg parallel_gripper)">
+    <maxwell_gripper name="gripper" parent="arm_wrist_roll" color="Orange">
+      <origin xyz="0 0 0" rpy="0 0 0" />
+    </maxwell_gripper>
+  </xacro:unless>
+  <!-- New Parallel Gripper -->
+  <xacro:if value="$(arg parallel_gripper)">
+    <maxwell_parallel_gripper name="gripper" parent="arm_wrist_roll" color="Orange">
+      <origin xyz="0 0 0" rpy="0 0 0" />
+    </maxwell_parallel_gripper>
+  </xacro:if>
   <!-- Head -->
   <maxwell_head name="head" parent="torso_link" color="Orange">
