Commit message: add upper arm roll joint

File: maxwell_defs/urdf/arm.urdf.xacro (robot description, xacro)
@@ -91,12 +91,45 @@
         <origin xyz="0 0 0" rpy="-1.57 0 0" />
         <geometry>
-          <mesh filename="package://maxwell_defs/meshes/arm_mx64_upper.stl" scale="1 1 1"/>
-        </geometry>
-        <material name="Black"/>
-      </visual>
-      <collision>
-        <origin xyz="0.08 0.0 0.0" rpy="0 0 0" />
-        <geometry>
-          <box size="0.204 0.053 0.044"/>
+          <mesh filename="package://maxwell_defs/meshes/sixdof_bracket2.stl" scale="0.001 0.001 0.001"/>
+        </geometry>
+        <material name="Black"/>
+      </visual>
+      <collision>
+        <origin xyz="0.0381 0.0 0.0" rpy="0 0 0" />
+        <geometry>
+          <box size="0.0762 0.053 0.044"/>
+        </geometry>
+      </collision>
+    </link>
+    <!-- Upper Arm Roll -->
+    <dynamixel_rx64_tilt parent="${name}_shoulder_lift_link" name="${name}_upperarm_roll_servo" color="Black">
+      <origin xyz="0.0839978 0 0" rpy="1.57 1.57 0"/>
+    </dynamixel_rx64_tilt>
+    <joint name="${name}_upperarm_roll_joint" type="revolute">
+      <origin xyz="0 0 0" rpy="-1.57 0 1.57"/>
+      <axis xyz="1 0 0"/>
+      <limit effort="30" velocity="0.524" lower="-3.14" upper="3.14" />
+      <parent link="${name}_upperarm_roll_servo_link"/>
+      <child link="${name}_upperarm_roll_link" />
+    </joint>
+    <link name="${name}_upperarm_roll_link">
+      <inertial>
+        <mass value="0.00001" />
+        <origin xyz="0 0 0" />
+        <inertia ixx="1.0" ixy="0.0" ixz="0.0"
+          iyy="1.0" iyz="0.0"
+          izz="1.0" />
+      </inertial>
+      <visual>
+        <origin xyz="0.074295 0 0" rpy="1.57 0 3.14" />
+        <geometry>
+          <mesh filename="package://maxwell_defs/meshes/sixdof_bracket1.stl" scale="0.001 0.001 0.001"/>
+        </geometry>
+        <material name="Black"/>
+      </visual>
+      <collision>
+        <origin xyz="0.0381 0.0 0.0" rpy="0 0 0" />
+        <geometry>
+          <box size="0.0762 0.053 0.044"/>
         </geometry>
       </collision>
@@ -104,8 +137,8 @@
     <!-- Elbow -->
     <joint name="${name}_elbow_flex_joint" type="revolute">
-      <origin xyz="0.16 0 0" rpy="0 0 0"/>
+      <origin xyz="0.074295 0 0" rpy="0 0 0"/>
       <axis xyz="0 1 0"/>
       <limit effort="30" velocity="0.524" lower="-1.57" upper="2.617" />
-      <parent link="${name}_shoulder_lift_link"/>
+      <parent link="${name}_upperarm_roll_link"/>
       <child link="${name}_elbow_flex_link" />
     </joint>

Commit message: reverse long and short brackets in urdf

File: maxwell_defs/urdf/arm.urdf.xacro (robot description, xacro)
@@ -91,5 +91,5 @@
         <origin xyz="0 0 0" rpy="-1.57 0 0" />
         <geometry>
-          <mesh filename="package://maxwell_defs/meshes/sixdof_bracket2.stl" scale="0.001 0.001 0.001"/>
+          <mesh filename="package://maxwell_defs/meshes/sixdof_bracket1.stl" scale="0.001 0.001 0.001"/>
         </geometry>
         <material name="Black"/>
@@ -104,5 +104,5 @@
     <!-- Upper Arm Roll -->
     <dynamixel_rx64_tilt parent="${name}_shoulder_lift_link" name="${name}_upperarm_roll_servo" color="Black">
-      <origin xyz="0.0839978 0 0" rpy="1.57 1.57 0"/>
+      <origin xyz="0.0712978 0 0" rpy="1.57 1.57 0"/>
     </dynamixel_rx64_tilt>
     <joint name="${name}_upperarm_roll_joint" type="revolute">
@@ -122,7 +122,7 @@
       </inertial>
       <visual>
-        <origin xyz="0.074295 0 0" rpy="1.57 0 3.14" />
-        <geometry>
-          <mesh filename="package://maxwell_defs/meshes/sixdof_bracket1.stl" scale="0.001 0.001 0.001"/>
+        <origin xyz="0.0869955 0 0" rpy="-1.57 0 3.14" />
+        <geometry>
+          <mesh filename="package://maxwell_defs/meshes/sixdof_bracket2.stl" scale="0.001 0.001 0.001"/>
         </geometry>
         <material name="Black"/>
@@ -137,5 +137,5 @@
     <!-- Elbow -->
     <joint name="${name}_elbow_flex_joint" type="revolute">
-      <origin xyz="0.074295 0 0" rpy="0 0 0"/>
+      <origin xyz="0.0869955 0 0" rpy="0 0 0"/>
       <axis xyz="0 1 0"/>
       <limit effort="30" velocity="0.524" lower="-1.57" upper="2.617" />

Commit message: updates for moveit

File: maxwell_defs/urdf/arm.urdf.xacro (robot description, xacro)
@@ -109,5 +109,5 @@
       <origin xyz="0 0 0" rpy="-1.57 0 1.57"/>
       <axis xyz="1 0 0"/>
-      <limit effort="30" velocity="0.524" lower="-3.14" upper="3.14" />
+      <limit effort="30" velocity="0.524" lower="-2" upper="2" />
       <parent link="${name}_upperarm_roll_servo_link"/>
       <child link="${name}_upperarm_roll_link" />

Commit message: update URDF for correctness, remove gripper_link

File: maxwell_defs/urdf/arm.urdf.xacro (robot description, xacro)
@@ -33,5 +33,5 @@
     <link name="${name}_link">
       <visual>
-        <origin xyz="0 0 -0.034" rpy="1.57 3.14 0" />
+        <origin xyz="0.01 0 -0.034" rpy="1.57 3.14 0" />
         <geometry>
           <mesh filename="package://maxwell_defs/meshes/arm_mount.stl" scale="0.001 0.001 0.001"/>
@@ -204,5 +204,5 @@
       <axis xyz="1 0 0" />
       <limit effort="30" velocity="0.785" lower="-2.617" upper="2.617"/>
-      <origin xyz="0.031 0 0" rpy="0 0 0" />
+      <origin xyz="0.041 0 0" rpy="0 0 0" />
       <parent link="${name}_wrist_flex_link"/>
       <child link="${name}_wrist_roll_link"/>

File: maxwell_defs/urdf/gripper.urdf.xacro (robot description, xacro)
@@ -44,19 +44,4 @@
       <origin xyz="0 -0.013 0" rpy="0 0 0"/>
     </ax12_F11_fixed>
-    <!-- Gripper Joint for Grasping -->
-    <joint name="${name}_joint" type="fixed">
-      <axis xyz="0 0 1" />
-      <origin xyz="0.15 0 -0.015" rpy="0 0 0"/>
-      <parent link="${parent}_link"/>
-      <child link="${name}_link"/>
-    </joint>
-    <link name="${name}_link">
-      <visual>
-        <origin xyz="0.0 0.0 0" rpy="0 0 0"/>
-        <geometry>
-          <sphere radius="0.0005"/>
-        </geometry>
-      </visual>
-    </link>
   </macro>
 </robot>
