Commit message: fix xacro warnings

File: maxwell_defs/urdf/arm.urdf.xacro (robot description, xacro)
@@ -1,8 +1,8 @@
 <?xml version="1.0"?>
-<robot>
+<robot xmlns:xacro="http://www.ros.org/wiki/xacro">
   <!-- standoffs -->
-  <macro name="standoffs" params="name parent length *origin">
+  <xacro:macro name="standoffs" params="name parent length *origin">
     <joint name="${name}_joint" type="fixed">
-      <insert_block name="origin" />
+      <xacro:insert_block name="origin" />
       <parent link="${parent}"/>
       <child link="${name}_link" />
@@ -23,9 +23,9 @@
       </collision>
     </link>
-  </macro>
+  </xacro:macro>
   <!-- cosmetics -->
-  <macro name="arm_mount" params="name parent *origin">
+  <xacro:macro name="arm_mount" params="name parent *origin">
     <joint name="${name}_joint" type="fixed">
-      <insert_block name="origin" />
+      <xacro:insert_block name="origin" />
       <parent link="${parent}"/>
       <child link="${name}_link" />
@@ -46,31 +46,31 @@
       </collision>
     </link>
-  </macro>
+  </xacro:macro>
   <!-- the actual arm -->
-  <macro name="maxwell_arm" params="name parent *origin">
+  <xacro:macro name="maxwell_arm" params="name parent *origin">
     <!-- Arm Link -->
     <joint name="${name}_base_joint" type="fixed">
-      <insert_block name="origin" />
+      <xacro:insert_block name="origin" />
       <parent link="${parent}"/>
       <child link="${name}_link"/>
     </joint>
     <link name="${name}_link"/>
-    <arm_mount name="${name}_left_mount" parent="${name}_link">
+    <xacro:arm_mount name="${name}_left_mount" parent="${name}_link">
       <origin xyz="-0.0611 0.0254 0" rpy="0 0 0"/>
-    </arm_mount>
-    <arm_mount name="${name}_right_mount" parent="${name}_link">
+    </xacro:arm_mount>
+    <xacro:arm_mount name="${name}_right_mount" parent="${name}_link">
       <origin xyz="-0.0611 ${-0.0254} 0" rpy="3.14 0 0"/>
-    </arm_mount>
+    </xacro:arm_mount>
     <!-- Shoulder pan -->
-    <dynamixel_rx64_pan parent="${name}_link" name="${name}_shoulder_pan_servo" color="Black">
+    <xacro:dynamixel_rx64_pan parent="${name}_link" name="${name}_shoulder_pan_servo" color="Black">
       <origin xyz="0 0 0" rpy="0 0 0"/>
-    </dynamixel_rx64_pan>
-    <rx64_side_revolute parent="${name}_shoulder_pan_servo_link" name="${name}_shoulder_pan" llimit="-1.57" ulimit="1.57" vlimit="0.524" color="Grey">
+    </xacro:dynamixel_rx64_pan>
+    <xacro:rx64_side_revolute parent="${name}_shoulder_pan_servo_link" name="${name}_shoulder_pan" llimit="-1.57" ulimit="1.57" vlimit="0.524" color="Grey">
       <origin xyz="0 0 0.0235" rpy="0 0 0"/>
-    </rx64_side_revolute>
+    </xacro:rx64_side_revolute>
     <!-- Shoulder lift -->
-    <dynamixel_rx64_tilt parent="${name}_shoulder_pan_link" name="${name}_shoulder_lift_servo" color="Black">
+    <xacro:dynamixel_rx64_tilt parent="${name}_shoulder_pan_link" name="${name}_shoulder_lift_servo" color="Black">
       <origin xyz="0 0 ${0.0611-0.013+0.0045}" rpy="0 -1.57 0"/>
-    </dynamixel_rx64_tilt>
+    </xacro:dynamixel_rx64_tilt>
     <joint name="${name}_shoulder_lift_joint" type="revolute">
       <origin xyz="0 0 0" rpy="0 1.57 0"/>
@@ -103,7 +103,7 @@
     </link>
     <!-- Upper Arm Roll -->
-    <dynamixel_rx64_tilt parent="${name}_shoulder_lift_link" name="${name}_upperarm_roll_servo" color="Black">
+    <xacro:dynamixel_rx64_tilt parent="${name}_shoulder_lift_link" name="${name}_upperarm_roll_servo" color="Black">
       <origin xyz="0.0712978 0 0" rpy="1.57 1.57 0"/>
-    </dynamixel_rx64_tilt>
+    </xacro:dynamixel_rx64_tilt>
     <joint name="${name}_upperarm_roll_joint" type="revolute">
       <origin xyz="0 0 0" rpy="-1.57 0 1.57"/>
@@ -194,10 +194,10 @@
     </link>
     <!-- Wrist flex -->
-    <dynamixel_rx64_tilt parent="${name}_forearm_link" name="${name}_wrist_flex_servo" color="Black">
+    <xacro:dynamixel_rx64_tilt parent="${name}_forearm_link" name="${name}_wrist_flex_servo" color="Black">
       <origin xyz="0.125 0 0" rpy="0 0 0"/>
-    </dynamixel_rx64_tilt>
-    <rx64_hinge parent="${name}_wrist_flex_servo_link" name="${name}_wrist_flex" llimit="-1.57" ulimit="1.57" vlimit="0.785" color="Grey">
+    </xacro:dynamixel_rx64_tilt>
+    <xacro:rx64_hinge parent="${name}_wrist_flex_servo_link" name="${name}_wrist_flex" llimit="-1.57" ulimit="1.57" vlimit="0.785" color="Grey">
       <origin xyz="0 0 0.0" rpy="0 0 0"/>
-    </rx64_hinge>
+    </xacro:rx64_hinge>
     <!-- Wrist roll -->
     <joint name="${name}_wrist_roll_joint" type="revolute">
@@ -230,4 +230,4 @@
       </collision>
     </link>
-  </macro>
+  </xacro:macro>
 </robot>

File: maxwell_defs/urdf/base.urdf.xacro (robot description, xacro)
@@ -2,18 +2,18 @@
 <robot xmlns:xacro="http://www.ros.org/wiki/xacro">
   <xacro:include filename="$(find maxwell_defs)/urdf/sensors/hokuyo_urg_laser.urdf.xacro" />
-  <property name="ground_clearance" value="0.0238" />
+  <xacro:property name="ground_clearance" value="0.0238" />
   <!-- simplified box collision geometry for base -->
-  <property name="wheels_offset_x" value="0.12065" />
-  <property name="wheel_offset_y" value="0.19304" />
-  <property name="wheel_length" value="0.02032" />
-  <property name="wheel_radius" value="0.06191" />
-  <property name="base_size_x" value="0.4064" />
-  <property name="base_size_y" value="0.4064" />
-  <property name="base_size_z" value="0.1310" />
+  <xacro:property name="wheels_offset_x" value="0.12065" />
+  <xacro:property name="wheel_offset_y" value="0.19304" />
+  <xacro:property name="wheel_length" value="0.02032" />
+  <xacro:property name="wheel_radius" value="0.06191" />
+  <xacro:property name="base_size_x" value="0.4064" />
+  <xacro:property name="base_size_y" value="0.4064" />
+  <xacro:property name="base_size_z" value="0.1310" />
   <!-- location of hokuyo laser -->
-  <property name="base_laser_x" value="0.0318" />
-  <property name="base_laser_z" value="0.1885" />
+  <xacro:property name="base_laser_x" value="0.0318" />
+  <xacro:property name="base_laser_z" value="0.1885" />
   <!-- define a wheel -->
-  <macro name="armadillo_wheel" params="suffix parent reflect color">
+  <xacro:macro name="armadillo_wheel" params="suffix parent reflect color">
     <joint name="${parent}_${suffix}_wheel_joint" type="continuous">
       <axis xyz="0 0 1" />
@@ -33,7 +33,7 @@
       </visual>
     </link>
-  </macro>
+  </xacro:macro>
   <!-- The xacro macro armadillo_base contains: base and wheels -->
-  <macro name="armadillo_base" params="name color">
+  <xacro:macro name="armadillo_base" params="name color">
     <link name="${name}_link">
       <visual>
@@ -52,10 +52,10 @@
     </link>
     <!-- base laser -->
-    <hokuyo_urg_laser name="${name}_laser" parent="${name}" >
+    <xacro:hokuyo_urg_laser name="${name}_laser" parent="${name}" >
       <origin xyz="${base_laser_x} 0 ${base_laser_z}" rpy="0 0 0" />
-    </hokuyo_urg_laser>
+    </xacro:hokuyo_urg_laser>
     <!-- drive wheels -->
-    <armadillo_wheel parent="${name}" suffix="l" reflect="1" color="${color}"/>
-    <armadillo_wheel parent="${name}" suffix="r" reflect="-1" color="${color}"/>
-  </macro>
+    <xacro:armadillo_wheel parent="${name}" suffix="l" reflect="1" color="${color}"/>
+    <xacro:armadillo_wheel parent="${name}" suffix="r" reflect="-1" color="${color}"/>
+  </xacro:macro>
 </robot>

File: maxwell_defs/urdf/gripper.urdf.xacro (robot description, xacro)
@@ -1,47 +1,47 @@
 <?xml version="1.0"?>
-<robot>
-  <macro name="maxwell_gripper" params="name parent color *origin">
-    <ax12_F6_fixed parent="${parent}_link" name="${name}_F6_1" color="Black">
+<robot xmlns:xacro="http://www.ros.org/wiki/xacro">
+  <xacro:macro name="maxwell_gripper" params="name parent color *origin">
+    <xacro:ax12_F6_fixed parent="${parent}_link" name="${name}_F6_1" color="Black">
       <origin xyz="${0.0381/2} 0.017 -0.014" rpy="0 0 0"/>
-    </ax12_F6_fixed>
-    <ax12_F6_fixed parent="${name}_F6_1_link" name="${name}_F6_2" color="Black">
+    </xacro:ax12_F6_fixed>
+    <xacro:ax12_F6_fixed parent="${name}_F6_1_link" name="${name}_F6_2" color="Black">
       <origin xyz="0.008 0.004 0" rpy="3.14 3.14 0"/>
-    </ax12_F6_fixed>
-    <ax12_F6_fixed parent="${parent}_link" name="${name}_F6_3" color="Black">
+    </xacro:ax12_F6_fixed>
+    <xacro:ax12_F6_fixed parent="${parent}_link" name="${name}_F6_3" color="Black">
       <origin xyz="${0.0381/2} -0.017 -0.014" rpy="3.14 0 0"/>
-    </ax12_F6_fixed>
-    <ax12_F6_fixed parent="${name}_F6_3_link" name="${name}_F6_4" color="Black">
+    </xacro:ax12_F6_fixed>
+    <xacro:ax12_F6_fixed parent="${name}_F6_3_link" name="${name}_F6_4" color="Black">
       <origin xyz="0.008 0.004 0" rpy="0 0 3.14"/>
-    </ax12_F6_fixed>
-    <ax12_side_fixed parent="${name}_F6_2_link" name="left_${name}_mount" color="Black">
+    </xacro:ax12_F6_fixed>
+    <xacro:ax12_side_fixed parent="${name}_F6_2_link" name="left_${name}_mount" color="Black">
       <origin xyz="-0.018 0.005 0" rpy="1.57 0 1.57"/>
-    </ax12_side_fixed>
-    <ax12_side_fixed parent="${name}_F6_4_link" name="right_${name}_mount" color="Black">
+    </xacro:ax12_side_fixed>
+    <xacro:ax12_side_fixed parent="${name}_F6_4_link" name="right_${name}_mount" color="Black">
       <origin xyz="-0.018 0.005 0" rpy="1.57 0 1.57"/>
-    </ax12_side_fixed>
-    <dynamixel_ax12_pan parent="left_${name}_mount_link" name="left_${name}_servo" color="Black">
+    </xacro:ax12_side_fixed>
+    <xacro:dynamixel_ax12_pan parent="left_${name}_mount_link" name="left_${name}_servo" color="Black">
       <origin xyz="0 0 -0.042" rpy="-1.57 1.57 0"/>
-    </dynamixel_ax12_pan>
-    <dynamixel_ax12_pan parent="right_${name}_mount_link" name="right_${name}_servo" color="Black">
+    </xacro:dynamixel_ax12_pan>
+    <xacro:dynamixel_ax12_pan parent="right_${name}_mount_link" name="right_${name}_servo" color="Black">
       <origin xyz="0 0 -0.042" rpy="1.57 1.57 0"/>
-    </dynamixel_ax12_pan>
-    <ax12_F1_revolute parent="left_${name}_servo_link" name="l_${name}" llimit="-1.57" ulimit="1.57" vlimit="0.5" color="${color}">
+    </xacro:dynamixel_ax12_pan>
+    <xacro:ax12_F1_revolute parent="left_${name}_servo_link" name="l_${name}" llimit="-1.57" ulimit="1.57" vlimit="0.5" color="${color}">
       <origin xyz="0 0 0" rpy="3.14 0 1.57"/>
-    </ax12_F1_revolute>
-    <ax12_F1_revolute parent="right_${name}_servo_link" name="r_${name}" llimit="-1.57" ulimit="1.57" vlimit="0.5" color="${color}">
+    </xacro:ax12_F1_revolute>
+    <xacro:ax12_F1_revolute parent="right_${name}_servo_link" name="r_${name}" llimit="-1.57" ulimit="1.57" vlimit="0.5" color="${color}">
       <origin xyz="0 0 0" rpy="0 0 -1.57"/>
-    </ax12_F1_revolute>
-    <ax12_F9_fixed parent="l_${name}_link" name="left_${name}_F9" color="Black">
+    </xacro:ax12_F1_revolute>
+    <xacro:ax12_F9_fixed parent="l_${name}_link" name="left_${name}_F9" color="Black">
       <origin xyz="0.0155 0.038 0" rpy="0 3.14 0"/>
-    </ax12_F9_fixed>
-    <ax12_F9_fixed parent="r_${name}_link" name="right_${name}_F9" color="Black">
+    </xacro:ax12_F9_fixed>
+    <xacro:ax12_F9_fixed parent="r_${name}_link" name="right_${name}_F9" color="Black">
       <origin xyz="0.0155 0.038 0" rpy="0 3.14 0"/>
-    </ax12_F9_fixed>
-    <ax12_F11_fixed parent="left_${name}_F9_link" name="left_${name}_finger" color="Grey">
+    </xacro:ax12_F9_fixed>
+    <xacro:ax12_F11_fixed parent="left_${name}_F9_link" name="left_${name}_finger" color="Grey">
       <origin xyz="0 -0.013 0 " rpy="0 0 0"/>
-    </ax12_F11_fixed>
-    <ax12_F11_fixed parent="right_${name}_F9_link" name="right_${name}_finger" color="Grey">
+    </xacro:ax12_F11_fixed>
+    <xacro:ax12_F11_fixed parent="right_${name}_F9_link" name="right_${name}_finger" color="Grey">
       <origin xyz="0 -0.013 0" rpy="0 0 0"/>
-    </ax12_F11_fixed>
-  </macro>
+    </xacro:ax12_F11_fixed>
+  </xacro:macro>
 </robot>

File: maxwell_defs/urdf/hardware/ax12.xacro (robot description, xacro)
@@ -1,9 +1,9 @@
 <?xml version="1.0"?>
-<robot>
-  <property name="AX12_WIDTH" value="0.038"/>
-  <property name="AX12_HEIGHT" value="0.0385"/>
-  <macro name="dynamixel_ax12_pan" params="parent name color *origin" >
-    <joint name="${name}_joint" type="fixed">
-      <insert_block name="origin" />
+<robot xmlns:xacro="http://www.ros.org/wiki/xacro">
+  <xacro:property name="AX12_WIDTH" value="0.038"/>
+  <xacro:property name="AX12_HEIGHT" value="0.0385"/>
+  <xacro:macro name="dynamixel_ax12_pan" params="parent name color *origin" >
+    <joint name="${name}_joint" type="fixed">
+      <xacro:insert_block name="origin" />
       <parent link="${parent}"/>
       <child link="${name}_link" />
@@ -31,8 +31,8 @@
       </collision>
     </link>
-  </macro>
-  <macro name="dynamixel_ax12_tilt" params="parent name color *origin" >
-    <joint name="${name}_joint" type="fixed">
-      <insert_block name="origin" />
+  </xacro:macro>
+  <xacro:macro name="dynamixel_ax12_tilt" params="parent name color *origin" >
+    <joint name="${name}_joint" type="fixed">
+      <xacro:insert_block name="origin" />
       <parent link="${parent}"/>
       <child link="${name}_link" />
@@ -60,8 +60,8 @@
       </collision>
     </link>
-  </macro>
-  <macro name="ax12_side_revolute" params="name parent llimit ulimit vlimit color *origin" >
+  </xacro:macro>
+  <xacro:macro name="ax12_side_revolute" params="name parent llimit ulimit vlimit color *origin" >
     <joint name="${name}_joint" type="revolute">
-      <insert_block name="origin" />
+      <xacro:insert_block name="origin" />
       <axis xyz="0 0 1"/>
       <limit effort="30" velocity="${vlimit}" lower="${llimit}" upper="${ulimit}" />
@@ -91,8 +91,8 @@
       </collision>
     </link>
-  </macro>
-  <macro name="ax12_side_fixed" params="parent name color *origin">
-    <joint name="${name}_joint" type="fixed">
-      <insert_block name="origin" />
+  </xacro:macro>
+  <xacro:macro name="ax12_side_fixed" params="parent name color *origin">
+    <joint name="${name}_joint" type="fixed">
+      <xacro:insert_block name="origin" />
       <parent link="${parent}"/>
       <child link="${name}_link" />
@@ -120,8 +120,8 @@
       </collision>
     </link>
-  </macro>
-  <macro name="ax12_hinge_revolute" params="parent name color llimit ulimit vlimit *origin">
+  </xacro:macro>
+  <xacro:macro name="ax12_hinge_revolute" params="parent name color llimit ulimit vlimit *origin">
     <joint name="${name}_joint" type="revolute">
-      <insert_block name="origin" />
+      <xacro:insert_block name="origin" />
        <axis xyz="0 1 0"/>
       <limit effort="30" velocity="${vlimit}" lower="${llimit}" upper="${ulimit}" />
@@ -151,8 +151,8 @@
       </collision>
     </link>
-  </macro>
-  <macro name="ax12_F1_revolute" params="name parent color llimit ulimit vlimit *origin">
+  </xacro:macro>
+  <xacro:macro name="ax12_F1_revolute" params="name parent color llimit ulimit vlimit *origin">
     <joint name="${name}_joint" type="revolute">
-      <insert_block name="origin" />
+      <xacro:insert_block name="origin" />
        <axis xyz="0 0 1"/>
       <limit effort="30" velocity="${vlimit}" lower="${llimit}" upper="${ulimit}" />
@@ -182,8 +182,8 @@
       </collision>
     </link>
-  </macro>
-  <macro name="ax12_F6_fixed" params="name parent color *origin">
-    <joint name="${name}_joint" type="fixed">
-      <insert_block name="origin" />
+  </xacro:macro>
+  <xacro:macro name="ax12_F6_fixed" params="name parent color *origin">
+    <joint name="${name}_joint" type="fixed">
+      <xacro:insert_block name="origin" />
       <parent link="${parent}"/>
       <child link="${name}_link" />
@@ -211,8 +211,8 @@
       </collision>
     </link>
-  </macro>
-  <macro name="ax12_F9_fixed" params="name parent color *origin">
-    <joint name="${name}_joint" type="fixed">
-      <insert_block name="origin" />
+  </xacro:macro>
+  <xacro:macro name="ax12_F9_fixed" params="name parent color *origin">
+    <joint name="${name}_joint" type="fixed">
+      <xacro:insert_block name="origin" />
       <parent link="${parent}"/>
       <child link="${name}_link" />
@@ -240,8 +240,8 @@
       </collision>
     </link>
-  </macro>
-  <macro name="ax12_F11_fixed" params="name parent color *origin">
-    <joint name="${name}_joint" type="fixed">
-      <insert_block name="origin" />
+  </xacro:macro>
+  <xacro:macro name="ax12_F11_fixed" params="name parent color *origin">
+    <joint name="${name}_joint" type="fixed">
+      <xacro:insert_block name="origin" />
       <parent link="${parent}"/>
       <child link="${name}_link" />
@@ -269,4 +269,4 @@
       </collision>
     </link>
-  </macro>
+  </xacro:macro>
 </robot>

File: maxwell_defs/urdf/hardware/rx28.xacro (robot description, xacro)
@@ -1,7 +1,7 @@
 <?xml version="1.0"?>
-<robot>
-  <macro name="dynamixel_rx28_pan" params="parent name color *origin" >
+<robot xmlns:xacro="http://www.ros.org/wiki/xacro">
+  <xacro:macro name="dynamixel_rx28_pan" params="parent name color *origin" >
     <joint name="${name}_joint" type="fixed">
-      <insert_block name="origin" />
+      <xacro:insert_block name="origin" />
       <parent link="${parent}"/>
       <child link="${name}_link" />
@@ -29,8 +29,8 @@
       </collision>
     </link>
-  </macro>
-  <macro name="dynamixel_rx28_tilt" params="parent name color *origin" >
+  </xacro:macro>
+  <xacro:macro name="dynamixel_rx28_tilt" params="parent name color *origin" >
     <joint name="${name}_joint" type="fixed">
-      <insert_block name="origin" />
+      <xacro:insert_block name="origin" />
       <parent link="${parent}"/>
       <child link="${name}_link" />
@@ -58,8 +58,8 @@
       </collision>
     </link>
-  </macro>
-  <macro name="rx28_side_revolute" params="parent name color llimit ulimit vlimit *origin">
+  </xacro:macro>
+  <xacro:macro name="rx28_side_revolute" params="parent name color llimit ulimit vlimit *origin">
     <joint name="${name}_joint" type="revolute">
-      <insert_block name="origin" />
+      <xacro:insert_block name="origin" />
        <axis xyz="1 0 0"/>
       <limit effort="30" velocity="${vlimit}" lower="${llimit}" upper="${ulimit}" />
@@ -89,8 +89,8 @@
       </collision>
     </link>
-  </macro>
-  <macro name="rx28_side_fixed" params="parent name color *origin">
+  </xacro:macro>
+  <xacro:macro name="rx28_side_fixed" params="parent name color *origin">
     <joint name="${name}_joint" type="fixed">
-      <insert_block name="origin" />
+      <xacro:insert_block name="origin" />
       <parent link="${parent}"/>
       <child link="${name}_link" />
@@ -118,8 +118,8 @@
       </collision>
     </link>
-  </macro>
-  <macro name="rx28_hinge" params="parent name color llimit ulimit vlimit *origin">
+  </xacro:macro>
+  <xacro:macro name="rx28_hinge" params="parent name color llimit ulimit vlimit *origin">
     <joint name="${name}_joint" type="revolute">
-      <insert_block name="origin" />
+      <xacro:insert_block name="origin" />
        <axis xyz="0 1 0"/>
       <limit effort="30" velocity="${vlimit}" lower="${llimit}" upper="${ulimit}" />
@@ -149,4 +149,4 @@
       </collision>
     </link>
-  </macro>
+  </xacro:macro>
 </robot>

File: maxwell_defs/urdf/hardware/rx64.xacro (robot description, xacro)
@@ -1,7 +1,7 @@
 <?xml version="1.0"?>
-<robot>
-  <macro name="dynamixel_rx64_pan" params="parent name color *origin" >
+<robot xmlns:xacro="http://www.ros.org/wiki/xacro">
+  <xacro:macro name="dynamixel_rx64_pan" params="parent name color *origin" >
     <joint name="${name}_joint" type="fixed">
-      <insert_block name="origin" />
+      <xacro:insert_block name="origin" />
       <parent link="${parent}"/>
       <child link="${name}_link" />
@@ -29,8 +29,8 @@
       </collision>
     </link>
-  </macro>
-  <macro name="dynamixel_rx64_tilt" params="parent name color *origin" >
+  </xacro:macro>
+  <xacro:macro name="dynamixel_rx64_tilt" params="parent name color *origin" >
     <joint name="${name}_joint" type="fixed">
-      <insert_block name="origin" />
+      <xacro:insert_block name="origin" />
       <parent link="${parent}"/>
       <child link="${name}_link" />
@@ -58,8 +58,8 @@
       </collision>
     </link>
-  </macro>
-  <macro name="rx64_side_revolute" params="parent name color llimit ulimit vlimit *origin">
+  </xacro:macro>
+  <xacro:macro name="rx64_side_revolute" params="parent name color llimit ulimit vlimit *origin">
     <joint name="${name}_joint" type="revolute">
-      <insert_block name="origin" />
+      <xacro:insert_block name="origin" />
        <axis xyz="0 0 1"/>
       <limit effort="30" velocity="${vlimit}" lower="${llimit}" upper="${ulimit}" />
@@ -89,8 +89,8 @@
       </collision>
     </link>
-  </macro>
-  <macro name="rx64_hinge" params="parent name color llimit ulimit vlimit *origin">
+  </xacro:macro>
+  <xacro:macro name="rx64_hinge" params="parent name color llimit ulimit vlimit *origin">
     <joint name="${name}_joint" type="revolute">
-      <insert_block name="origin" />
+      <xacro:insert_block name="origin" />
        <axis xyz="0 1 0"/>
       <limit effort="30" velocity="${vlimit}" lower="${llimit}" upper="${ulimit}" />
@@ -120,4 +120,4 @@
       </collision>
     </link>
-  </macro>
+  </xacro:macro>
 </robot>
