Commit message: fix xacro warnings

File: maxwell_defs/urdf/head.urdf.xacro (robot description, xacro)
@@ -1,8 +1,8 @@
 <?xml version="1.0"?>
-<robot>
+<robot xmlns:xacro="http://www.ros.org/wiki/xacro">
   <!-- cosmetics -->
-  <macro name="head_mount" params="name parent *origin">
+  <xacro:macro name="head_mount" params="name parent *origin">
     <joint name="${name}_joint" type="fixed">
-      <insert_block name="origin" />
+      <xacro:insert_block name="origin" />
       <parent link="${parent}"/>
       <child link="${name}_link" />
@@ -23,39 +23,39 @@
       </collision>
     </link>
-  </macro>
+  </xacro:macro>
   <!-- origin is center of head tilt rotation -->
-  <macro name="maxwell_head" params="name parent color *origin">
+  <xacro:macro name="maxwell_head" params="name parent color *origin">
     <joint name="${name}_joint" type="fixed">
-      <insert_block name="origin" />
+      <xacro:insert_block name="origin" />
       <parent link="${parent}"/>
       <child link="${name}_link"/>
     </joint>
     <link name="${name}_link"/>
-    <head_mount name="${name}_left_mount" parent="${name}_link">
+    <xacro:head_mount name="${name}_left_mount" parent="${name}_link">
       <origin xyz="0 0.01905 0" rpy="0 0 0"/>
-    </head_mount>
-    <head_mount name="${name}_right_mount" parent="${name}_link">
+    </xacro:head_mount>
+    <xacro:head_mount name="${name}_right_mount" parent="${name}_link">
       <origin xyz="0 ${-0.01905-0.003175} 0" rpy="0 0 0"/>
-    </head_mount>
+    </xacro:head_mount>
     <!-- Head pan -->
-    <dynamixel_ax12_pan parent="${name}_link" name="${name}_pan_servo" color="Black">
+    <xacro:dynamixel_ax12_pan parent="${name}_link" name="${name}_pan_servo" color="Black">
       <origin xyz="0.010 0 0.0254" rpy="0 0 0"/>
-    </dynamixel_ax12_pan>
-    <ax12_side_revolute parent="${name}_pan_servo_link" name="${name}_pan" llimit="-2.617" ulimit="2.617" vlimit="1.0" color="${color}">
+    </xacro:dynamixel_ax12_pan>
+    <xacro:ax12_side_revolute parent="${name}_pan_servo_link" name="${name}_pan" llimit="-2.617" ulimit="2.617" vlimit="1.0" color="${color}">
       <origin xyz="0 0 ${AX12_WIDTH/2}" rpy="0 0 0"/>
-    </ax12_side_revolute>
-    <ax12_side_fixed parent="${name}_pan_servo_link" name="${name}_tilt_left_side" color="Black">
+    </xacro:ax12_side_revolute>
+    <xacro:ax12_side_fixed parent="${name}_pan_servo_link" name="${name}_tilt_left_side" color="Black">
       <origin xyz="-0.015 ${-AX12_WIDTH/2} 0" rpy="1.57 0 0"/>
-    </ax12_side_fixed>
-    <ax12_side_fixed parent="${name}_pan_servo_link" name="${name}_tilt_right_side" color="Black">
+    </xacro:ax12_side_fixed>
+    <xacro:ax12_side_fixed parent="${name}_pan_servo_link" name="${name}_tilt_right_side" color="Black">
       <origin xyz="-0.015 ${AX12_WIDTH/2} 0" rpy="-1.57 0 0"/>
-    </ax12_side_fixed>
+    </xacro:ax12_side_fixed>
     <!-- Head tilt -->
-    <dynamixel_ax12_tilt parent="${name}_pan_link" name="${name}_tilt_servo" color="Black">
+    <xacro:dynamixel_ax12_tilt parent="${name}_pan_link" name="${name}_tilt_servo" color="Black">
       <origin xyz="0 0 ${AX12_HEIGHT+0.003}" rpy="0 0 0"/>
-    </dynamixel_ax12_tilt>
-    <ax12_hinge_revolute parent="${name}_tilt_servo_link" name="${name}_tilt" llimit="-1.57" ulimit="1.57" vlimit="1.0" color="${color}">
+    </xacro:dynamixel_ax12_tilt>
+    <xacro:ax12_hinge_revolute parent="${name}_tilt_servo_link" name="${name}_tilt" llimit="-1.57" ulimit="1.57" vlimit="1.0" color="${color}">
      <origin xyz="0 0 0" rpy="0 0 0"/>
-    </ax12_hinge_revolute>
-  </macro>
+    </xacro:ax12_hinge_revolute>
+  </xacro:macro>
 </robot>

File: maxwell_defs/urdf/maxwell.urdf.xacro (robot description, xacro)
@@ -15,9 +15,9 @@
   <xacro:include filename="$(find maxwell_defs)/urdf/materials.urdf.xacro" />
   <!-- Now we can start using the macros included above to define the actual Maxwell -->
-  <armadillo_base name="base" color="Orange"/>
+  <xacro:armadillo_base name="base" color="Orange"/>
   <!-- Add Torso Upright -->
-  <maxwell_torso name="torso" parent="base_link">
+  <xacro:maxwell_torso name="torso" parent="base_link">
     <origin xyz="-0.00635 0 ${base_size_z+arm_height}" rpy="0 0 0"/>
-  </maxwell_torso>
+  </xacro:maxwell_torso>
   <!-- Live joint between torso and arm -->
   <joint name="arm_lift_joint" type="prismatic">
@@ -30,25 +30,25 @@
   <link name="arm_lift_link"/>
   <!-- Arm -->
-  <maxwell_arm name="arm" parent="arm_lift_link">
+  <xacro:maxwell_arm name="arm" parent="arm_lift_link">
     <origin xyz="0.0611 0 0" rpy="0 0 0"/>
-  </maxwell_arm>
+  </xacro:maxwell_arm>
   <!-- Older Two Finger Gripper -->
   <xacro:unless value="$(arg parallel_gripper)">
-    <maxwell_gripper name="gripper" parent="arm_wrist_roll" color="Orange">
+    <xacro:maxwell_gripper name="gripper" parent="arm_wrist_roll" color="Orange">
       <origin xyz="0 0 0" rpy="0 0 0" />
-    </maxwell_gripper>
+    </xacro:maxwell_gripper>
   </xacro:unless>
   <!-- New Parallel Gripper -->
   <xacro:if value="$(arg parallel_gripper)">
-    <maxwell_parallel_gripper name="gripper" parent="arm_wrist_roll" color="Orange">
+    <xacro:maxwell_parallel_gripper name="gripper" parent="arm_wrist_roll" color="Orange">
       <origin xyz="0 0 0" rpy="0 0 0" />
-    </maxwell_parallel_gripper>
+    </xacro:maxwell_parallel_gripper>
   </xacro:if>
   <!-- Head -->
-  <maxwell_head name="head" parent="torso_link" color="Orange">
+  <xacro:maxwell_head name="head" parent="torso_link" color="Orange">
     <origin xyz="0 0 ${column_height-arm_height}" rpy="0 0 0"/>
-  </maxwell_head>
-  <xtion_camera name="head_camera" parent="head_tilt_link">
+  </xacro:maxwell_head>
+  <xacro:xtion_camera name="head_camera" parent="head_tilt_link">
     <origin xyz="0 0 0.026" rpy="0 0 0"/>
-  </xtion_camera>
+  </xacro:xtion_camera>
 </robot>

File: maxwell_defs/urdf/parallel_gripper.urdf.xacro (robot description, xacro)
@@ -1,14 +1,14 @@
 <?xml version="1.0"?>
-<robot>
-  <property name="parallel_gripper_width" value="0.112" />
-  <property name="parallel_gripper_length" value="0.114" />
-  <property name="parallel_gripper_height" value="0.044" />
-  <property name="parallel_gripper_finger_width" value="0.010" />
-  <property name="parallel_gripper_finger_length" value="0.0508" />
-  <property name="parallel_gripper_finger_height" value="0.027" />
-  <macro name="maxwell_parallel_gripper_finger" params="suffix parent reflect color *origin">
+<robot xmlns:xacro="http://www.ros.org/wiki/xacro">
+  <xacro:property name="parallel_gripper_width" value="0.112" />
+  <xacro:property name="parallel_gripper_length" value="0.114" />
+  <xacro:property name="parallel_gripper_height" value="0.044" />
+  <xacro:property name="parallel_gripper_finger_width" value="0.010" />
+  <xacro:property name="parallel_gripper_finger_length" value="0.0508" />
+  <xacro:property name="parallel_gripper_finger_height" value="0.027" />
+  <xacro:macro name="maxwell_parallel_gripper_finger" params="suffix parent reflect color *origin">
     <link name="${parent}_${suffix}_finger_link">
       <visual>
-        <insert_block name="origin" />
+        <xacro:insert_block name="origin" />
         <geometry>
           <box size="${parallel_gripper_finger_length} ${parallel_gripper_finger_width} ${parallel_gripper_finger_height}" />
@@ -24,6 +24,6 @@
       <child link="${parent}_${suffix}_finger_link"/>
     </joint>
-  </macro>
-  <macro name="maxwell_parallel_gripper" params="name parent color *origin">
+  </xacro:macro>
+  <xacro:macro name="maxwell_parallel_gripper" params="name parent color *origin">
     <link name="${name}_link">
       <visual>
@@ -40,10 +40,10 @@
       <child link="${name}_link"/>
     </joint>
-    <maxwell_parallel_gripper_finger parent="${name}" suffix="l" reflect="1" color="Orange" >
+    <xacro:maxwell_parallel_gripper_finger parent="${name}" suffix="l" reflect="1" color="Orange" >
       <origin xyz="${parallel_gripper_length/2} 0 0" rpy="0 0 0"/>
-    </maxwell_parallel_gripper_finger>
-    <maxwell_parallel_gripper_finger parent="${name}" suffix="r" reflect="-1" color="Orange" >
+    </xacro:maxwell_parallel_gripper_finger>
+    <xacro:maxwell_parallel_gripper_finger parent="${name}" suffix="r" reflect="-1" color="Orange" >
       <origin xyz="${parallel_gripper_length/2} 0 0" rpy="0 0 0"/>
-    </maxwell_parallel_gripper_finger>
-  </macro>
+    </xacro:maxwell_parallel_gripper_finger>
+  </xacro:macro>
 </robot>

File: maxwell_defs/urdf/sensors/hokuyo_urg_laser.urdf.xacro (robot description, xacro)
@@ -1,8 +1,8 @@
 <?xml version="1.0"?>
-<robot>
-  <macro name="hokuyo_urg_laser" params="name parent *origin">
+<robot xmlns:xacro="http://www.ros.org/wiki/xacro">
+  <xacro:macro name="hokuyo_urg_laser" params="name parent *origin">
     <joint name="${name}_joint" type="fixed">
       <axis xyz="0 1 0" />
-      <insert_block name="origin" />
+      <xacro:insert_block name="origin" />
       <parent link="${parent}_link"/>
       <child link="${name}_link"/>
@@ -28,4 +28,4 @@
       </collision>
     </link>
-  </macro>
+  </xacro:macro>
 </robot>

File: maxwell_defs/urdf/sensors/kinect_camera.urdf.xacro (robot description, xacro)
@@ -1,7 +1,7 @@
 <?xml version="1.0"?>
-<robot>
-  <macro name="kinect_camera" params="name parent *origin">
+<robot xmlns:xacro="http://www.ros.org/wiki/xacro">
+  <xacro:macro name="kinect_camera" params="name parent *origin">
     <joint name="${name}_frame_joint" type="fixed">
-      <insert_block name="origin" />
+      <xacro:insert_block name="origin" />
       <parent link="${parent}"/>
       <child link="${name}_frame"/>
@@ -65,4 +65,4 @@
     </joint>
     <link name="${name}_rgb_optical_frame"/>
-  </macro>
+  </xacro:macro>
 </robot>

File: maxwell_defs/urdf/sensors/xtion_camera.xacro (robot description, xacro)
@@ -1,7 +1,7 @@
 <?xml version="1.0"?>
-<robot>
-  <macro name="xtion_camera" params="name parent *origin">
+<robot xmlns:xacro="http://www.ros.org/wiki/xacro">
+  <xacro:macro name="xtion_camera" params="name parent *origin">
     <joint name="${name}_frame_joint" type="fixed">
-      <insert_block name="origin" />
+      <xacro:insert_block name="origin" />
       <parent link="${parent}"/>
       <child link="${name}_frame"/>
@@ -64,4 +64,4 @@
     </joint>
     <link name="${name}_rgb_optical_frame"/>
-  </macro>
+  </xacro:macro>
 </robot>

File: maxwell_defs/urdf/torso.urdf.xacro (robot description, xacro)
@@ -1,7 +1,7 @@
 <?xml version="1.0"?>
-<robot>
-  <macro name="maxwell_torso" params="name parent *origin">
+<robot xmlns:xacro="http://www.ros.org/wiki/xacro">
+  <xacro:macro name="maxwell_torso" params="name parent *origin">
     <joint name="${name}_joint" type="fixed">
-      <insert_block name="origin" />
+      <xacro:insert_block name="origin" />
       <parent link="${parent}"/>
       <child link="${name}_link"/>
@@ -42,4 +42,4 @@
       </collision>
     </link>
-  </macro>
+  </xacro:macro>
 </robot>
