Commit message: fixup urdf after rename

File: maxwell/urdf/arm.urdf.xacro (robot description, xacro)
@@ -35,5 +35,5 @@
         <origin xyz="0.01 0 -0.034" rpy="1.57 3.14 0" />
         <geometry>
-          <mesh filename="package://maxwell_defs/meshes/arm_mount.stl" scale="0.001 0.001 0.001"/>
+          <mesh filename="package://maxwell/meshes/arm_mount.stl" scale="0.001 0.001 0.001"/>
         </geometry>
         <material name="Black"/>
@@ -91,5 +91,5 @@
         <origin xyz="0 0 0" rpy="-1.57 0 0" />
         <geometry>
-          <mesh filename="package://maxwell_defs/meshes/sixdof_bracket1.stl" scale="0.001 0.001 0.001"/>
+          <mesh filename="package://maxwell/meshes/sixdof_bracket1.stl" scale="0.001 0.001 0.001"/>
         </geometry>
         <material name="Black"/>
@@ -124,5 +124,5 @@
         <origin xyz="0.0869955 0 0" rpy="-1.57 0 3.14" />
         <geometry>
-          <mesh filename="package://maxwell_defs/meshes/sixdof_bracket2.stl" scale="0.001 0.001 0.001"/>
+          <mesh filename="package://maxwell/meshes/sixdof_bracket2.stl" scale="0.001 0.001 0.001"/>
         </geometry>
         <material name="Black"/>
@@ -154,5 +154,5 @@
         <origin xyz=" 0 0 0 " rpy="1.57 -1.57 0" />
         <geometry>
-          <mesh filename="package://maxwell_defs/meshes/rx64.stl" scale="1 1 1"/>
+          <mesh filename="package://maxwell/meshes/rx64.stl" scale="1 1 1"/>
         </geometry>
         <material name="Black"/>
@@ -182,5 +182,5 @@
         <origin xyz="0 0 0" rpy="-1.57 0 0" />
         <geometry>
-          <mesh filename="package://maxwell_defs/meshes/arm_mx64_forearm.stl" scale="1 1 1"/>
+          <mesh filename="package://maxwell/meshes/arm_mx64_forearm.stl" scale="1 1 1"/>
         </geometry>
         <material name="Black"/>
@@ -219,5 +219,5 @@
         <origin xyz="${0.0381/2} 0 0" rpy="0 0 1.57" />
         <geometry>
-          <mesh filename="package://maxwell_defs/meshes/ax12.stl" scale="0.001 0.001 0.001"/>
+          <mesh filename="package://maxwell/meshes/ax12.stl" scale="0.001 0.001 0.001"/>
         </geometry>
         <material name="Black"/>

File: maxwell/urdf/base.urdf.xacro (robot description, xacro)
@@ -1,5 +1,5 @@
 <?xml version="1.0"?>
 <robot xmlns:xacro="http://www.ros.org/wiki/xacro">
-  <xacro:include filename="$(find maxwell_defs)/urdf/sensors/hokuyo_urg_laser.urdf.xacro" />
+  <xacro:include filename="$(find maxwell)/urdf/sensors/hokuyo_urg_laser.urdf.xacro" />
   <xacro:property name="ground_clearance" value="0.0238" />
   <!-- simplified box collision geometry for base -->
@@ -40,5 +40,5 @@
         <origin xyz="0 0 ${ground_clearance}" rpy="0 0 0" />
         <geometry>
-          <mesh filename="package://maxwell_defs/meshes/base.stl"  />
+          <mesh filename="package://maxwell/meshes/base.stl"  />
         </geometry>
         <material name="Black" />

File: maxwell/urdf/hardware/ax12.xacro (robot description, xacro)
@@ -20,5 +20,5 @@
         <origin xyz=" 0 0 0 " rpy="1.57 0 1.57" />
         <geometry>
-          <mesh filename="package://maxwell_defs/meshes/ax12.stl" scale="0.001 0.001 0.001"/>
+          <mesh filename="package://maxwell/meshes/ax12.stl" scale="0.001 0.001 0.001"/>
         </geometry>
         <material name="${color}"/>
@@ -49,5 +49,5 @@
         <origin xyz=" 0 0 0 " rpy="0 0 0" />
         <geometry>
-          <mesh filename="package://maxwell_defs/meshes/ax12.stl" scale="0.001 0.001 0.001"/>
+          <mesh filename="package://maxwell/meshes/ax12.stl" scale="0.001 0.001 0.001"/>
         </geometry>
         <material name="${color}"/>
@@ -80,5 +80,5 @@
         <origin xyz=" 0 0 0 " rpy="3.14 0 0" />
         <geometry>
-          <mesh filename="package://maxwell_defs/meshes/F3.stl" scale="0.001 0.001 0.001"/>
+          <mesh filename="package://maxwell/meshes/F3.stl" scale="0.001 0.001 0.001"/>
         </geometry>
         <material name="${color}"/>
@@ -109,5 +109,5 @@
         <origin xyz=" 0 0 0 " rpy="0 0 0" />
         <geometry>
-          <mesh filename="package://maxwell_defs/meshes/F3.stl" scale="0.001 0.001 0.001"/>
+          <mesh filename="package://maxwell/meshes/F3.stl" scale="0.001 0.001 0.001"/>
         </geometry>
         <material name="${color}"/>
@@ -140,5 +140,5 @@
         <origin xyz=" 0 0 0 " rpy="0 0 0" />
         <geometry>
-          <mesh filename="package://maxwell_defs/meshes/F2.stl" scale="0.001 0.001 0.001"/>
+          <mesh filename="package://maxwell/meshes/F2.stl" scale="0.001 0.001 0.001"/>
         </geometry>
         <material name="${color}"/>
@@ -171,5 +171,5 @@
         <origin xyz=" 0 0 0 " rpy="3.14 0 0" />
         <geometry>
-          <mesh filename="package://maxwell_defs/meshes/F1.stl" scale="1 1 1"/>
+          <mesh filename="package://maxwell/meshes/F1.stl" scale="1 1 1"/>
         </geometry>
         <material name="${color}"/>
@@ -200,5 +200,5 @@
         <origin xyz=" 0 0 0 " rpy="3.14 0 0" />
         <geometry>
-          <mesh filename="package://maxwell_defs/meshes/F6.stl" scale="1 1 1"/>
+          <mesh filename="package://maxwell/meshes/F6.stl" scale="1 1 1"/>
         </geometry>
         <material name="${color}"/>
@@ -229,5 +229,5 @@
         <origin xyz="0 0 0" rpy="0 0 0" />
         <geometry>
-          <mesh filename="package://maxwell_defs/meshes/F9.stl" scale="1 1 1"/>
+          <mesh filename="package://maxwell/meshes/F9.stl" scale="1 1 1"/>
         </geometry>
         <material name="${color}"/>
@@ -258,5 +258,5 @@
         <origin xyz="0 0 0" rpy="0 0 0" />
         <geometry>
-          <mesh filename="package://maxwell_defs/meshes/F11.stl" scale="1 1 1"/>
+          <mesh filename="package://maxwell/meshes/F11.stl" scale="1 1 1"/>
         </geometry>
         <material name="${color}"/>

File: maxwell/urdf/hardware/rx28.xacro (robot description, xacro)
@@ -18,5 +18,5 @@
         <origin xyz=" 0 0 0 " rpy="0 0 -1.57" />
         <geometry>
-          <mesh filename="package://maxwell_defs/meshes/rx28.stl" scale="1 1 1"/>
+          <mesh filename="package://maxwell/meshes/rx28.stl" scale="1 1 1"/>
         </geometry>
         <material name="${color}"/>
@@ -47,5 +47,5 @@
         <origin xyz=" 0 0 0 " rpy="1.57 1.57 0" />
         <geometry>
-          <mesh filename="package://maxwell_defs/meshes/rx28.stl" scale="1 1 1"/>
+          <mesh filename="package://maxwell/meshes/rx28.stl" scale="1 1 1"/>
         </geometry>
         <material name="${color}"/>
@@ -78,5 +78,5 @@
         <origin xyz=" 0 0 0 " rpy="-1.57 -1.57 0" />
         <geometry>
-          <mesh filename="package://maxwell_defs/meshes/rx28-side-bracket.stl" scale="1 1 1"/>
+          <mesh filename="package://maxwell/meshes/rx28-side-bracket.stl" scale="1 1 1"/>
         </geometry>
         <material name="${color}"/>
@@ -107,5 +107,5 @@
         <origin xyz=" 0 0 0 " rpy="1.57 1.57 0" />
         <geometry>
-          <mesh filename="package://maxwell_defs/meshes/rx28-side-bracket.stl" scale="1 1 1"/>
+          <mesh filename="package://maxwell/meshes/rx28-side-bracket.stl" scale="1 1 1"/>
         </geometry>
         <material name="${color}"/>
@@ -138,5 +138,5 @@
         <origin xyz="0 0 0" rpy="0 0 -1.57" />
         <geometry>
-          <mesh filename="package://maxwell_defs/meshes/rx28-hinge-bracket.stl" scale="1 1 1"/>
+          <mesh filename="package://maxwell/meshes/rx28-hinge-bracket.stl" scale="1 1 1"/>
         </geometry>
         <material name="${color}"/>

File: maxwell/urdf/hardware/rx64.xacro (robot description, xacro)
@@ -18,5 +18,5 @@
         <origin xyz=" 0 0 0 " rpy="0 0 -1.57" />
         <geometry>
-          <mesh filename="package://maxwell_defs/meshes/rx64.stl" scale="1 1 1"/>
+          <mesh filename="package://maxwell/meshes/rx64.stl" scale="1 1 1"/>
         </geometry>
         <material name="${color}"/>
@@ -47,5 +47,5 @@
         <origin xyz=" 0 0 0 " rpy="1.57 1.57 0" />
         <geometry>
-          <mesh filename="package://maxwell_defs/meshes/rx64.stl" scale="1 1 1"/>
+          <mesh filename="package://maxwell/meshes/rx64.stl" scale="1 1 1"/>
         </geometry>
         <material name="${color}"/>
@@ -78,5 +78,5 @@
         <origin xyz=" 0 0 0 " rpy="1.57 0 0" />
         <geometry>
-          <mesh filename="package://maxwell_defs/meshes/rx64-side-bracket.stl" scale="1 1 1"/>
+          <mesh filename="package://maxwell/meshes/rx64-side-bracket.stl" scale="1 1 1"/>
         </geometry>
         <material name="${color}"/>
@@ -109,5 +109,5 @@
         <origin xyz="0 0 0" rpy="0 0 -1.57" />
         <geometry>
-          <mesh filename="package://maxwell_defs/meshes/rx64-hinge-bracket.stl" scale="1 1 1"/>
+          <mesh filename="package://maxwell/meshes/rx64-hinge-bracket.stl" scale="1 1 1"/>
         </geometry>
         <material name="${color}"/>

File: maxwell/urdf/head.urdf.xacro (robot description, xacro)
@@ -12,5 +12,5 @@
         <origin xyz="0 0 0" rpy="-1.57 3.14 0" />
         <geometry>
-          <mesh filename="package://maxwell_defs/meshes/head_mount.stl" scale="1 1 1"/>
+          <mesh filename="package://maxwell/meshes/head_mount.stl" scale="1 1 1"/>
         </geometry>
         <material name="Black"/>

File: maxwell/urdf/maxwell.urdf.xacro (robot description, xacro)
@@ -3,15 +3,15 @@
   <xacro:property name="arm_height" value="0.6604"/> <!-- deck to arm_link at max height-->
   <xacro:property name="column_height" value="1.172775" /> <!-- deck to top of 80/20 -->
-  <xacro:include filename="$(find maxwell_defs)/urdf/hardware/ax12.xacro" />
-  <xacro:include filename="$(find maxwell_defs)/urdf/hardware/rx64.xacro" />
-  <xacro:include filename="$(find maxwell_defs)/urdf/sensors/xtion_camera.xacro" />
+  <xacro:include filename="$(find maxwell)/urdf/hardware/ax12.xacro" />
+  <xacro:include filename="$(find maxwell)/urdf/hardware/rx64.xacro" />
+  <xacro:include filename="$(find maxwell)/urdf/sensors/xtion_camera.xacro" />
   <!-- The following included files set up definitions of parts of the robot body -->
-  <xacro:include filename="$(find maxwell_defs)/urdf/base.urdf.xacro" />
-  <xacro:include filename="$(find maxwell_defs)/urdf/torso.urdf.xacro" />
-  <xacro:include filename="$(find maxwell_defs)/urdf/arm.urdf.xacro" />
-  <xacro:include filename="$(find maxwell_defs)/urdf/gripper.urdf.xacro" />
-  <xacro:include filename="$(find maxwell_defs)/urdf/parallel_gripper.urdf.xacro" />
-  <xacro:include filename="$(find maxwell_defs)/urdf/head.urdf.xacro" />
-  <xacro:include filename="$(find maxwell_defs)/urdf/materials.urdf.xacro" />
+  <xacro:include filename="$(find maxwell)/urdf/base.urdf.xacro" />
+  <xacro:include filename="$(find maxwell)/urdf/torso.urdf.xacro" />
+  <xacro:include filename="$(find maxwell)/urdf/arm.urdf.xacro" />
+  <xacro:include filename="$(find maxwell)/urdf/gripper.urdf.xacro" />
+  <xacro:include filename="$(find maxwell)/urdf/parallel_gripper.urdf.xacro" />
+  <xacro:include filename="$(find maxwell)/urdf/head.urdf.xacro" />
+  <xacro:include filename="$(find maxwell)/urdf/materials.urdf.xacro" />
   <!-- Now we can start using the macros included above to define the actual Maxwell -->
   <xacro:armadillo_base name="base" color="Orange"/>
@@ -33,16 +33,8 @@
     <origin xyz="0.0611 0 0" rpy="0 0 0"/>
   </xacro:maxwell_arm>
-  <!-- Older Two Finger Gripper -->
-  <xacro:unless value="$(arg parallel_gripper)">
-    <xacro:maxwell_gripper name="gripper" parent="arm_wrist_roll" color="Orange">
-      <origin xyz="0 0 0" rpy="0 0 0" />
-    </xacro:maxwell_gripper>
-  </xacro:unless>
   <!-- New Parallel Gripper -->
-  <xacro:if value="$(arg parallel_gripper)">
-    <xacro:maxwell_parallel_gripper name="gripper" parent="arm_wrist_roll" color="Orange">
-      <origin xyz="0 0 0" rpy="0 0 0" />
-    </xacro:maxwell_parallel_gripper>
-  </xacro:if>
+  <xacro:maxwell_parallel_gripper name="gripper" parent="arm_wrist_roll" color="Orange">
+    <origin xyz="0 0 0" rpy="0 0 0" />
+  </xacro:maxwell_parallel_gripper>
   <!-- Head -->
   <xacro:maxwell_head name="head" parent="torso_link" color="Orange">

File: maxwell/urdf/sensors/kinect_camera.urdf.xacro (robot description, xacro)
@@ -12,5 +12,5 @@
         <!--origin xyz="-0.03 -0.07 0" rpy="0 0 -1.57"-->
         <geometry>
-          <mesh filename="package://maxwell_defs/meshes/kinect.stl" />
+          <mesh filename="package://maxwell/meshes/kinect.stl" />
         </geometry>
         <material name="Black" />

File: maxwell/urdf/sensors/xtion_camera.xacro (robot description, xacro)
@@ -11,5 +11,5 @@
         <origin xyz="0 0 0" rpy="0 0 -1.57" />
         <geometry>
-          <mesh filename="package://maxwell_defs/meshes/xtion.stl" scale="0.001 0.001 0.001"/>
+          <mesh filename="package://maxwell/meshes/xtion.stl" scale="0.001 0.001 0.001"/>
         </geometry>
         <material name="Black" />

File: maxwell/urdf/torso.urdf.xacro (robot description, xacro)
@@ -31,5 +31,5 @@
         <origin xyz="-0.05 -0.0127 -0.560" rpy="0 0 3.14" />
         <geometry>
-          <mesh filename="package://maxwell_defs/meshes/FA-35-TR.stl" scale="0.001 0.001 0.001"/>
+          <mesh filename="package://maxwell/meshes/FA-35-TR.stl" scale="0.001 0.001 0.001"/>
         </geometry>
         <material name="Grey"/>
